Commit message: reconbot_mods

File: reconbot_description/urdf/reconbot_mobile_base_gazebo.xacro (robot description, xacro)
@@ -41,9 +41,19 @@
     </gazebo>
     <gazebo>
-        <plugin name="buoyancy_plugin" filename="libuuv_underwater_buoyancy_plugin.so">
-            <link_name>base_footprint</link_name>
-            <fluid_density>997</fluid_density>
-            <surface_height>0.0</surface_height>
+        <plugin name="buoyancy_plugin" filename="libBuoyancyPlugin.so">
+        <fluid_density>997</fluid_density>
+        <link name="base_link">
+            <center_of_buoyancy>-0.0 0.0 0</center_of_buoyancy>
+            <volume>0.04203149</volume>
             <neutrally_buoyant>true</neutrally_buoyant>
+        </link>
+        </plugin>
+    </gazebo>
+    <gazebo>
+        <plugin name="hydrodynamics_plugin" filename="libHydrodynamicsPlugin.so">
+        <link_name>base_link</link_name>
+        <fluid_density>997</fluid_density>
+        <linear_drag_coefficients>10.0 10.0 10.0</linear_drag_coefficients>
+        <angular_drag_coefficients>1.0 1.0 1.0</angular_drag_coefficients>
         </plugin>
     </gazebo>
