Commit message: gazebo add

File: reconbot_description/urdf/reconbot_mobile_base.xacro (robot description, xacro)
@@ -1,4 +1,4 @@
 <?xml version="1.0"?>
-<robot name="gr2" xmlns:xacro="http://www.ros.org/wiki/xacro">
+<robot xmlns:xacro="http://www.ros.org/wiki/xacro">
     <link name="base_footprint" />
     <link name="base_link">
@@ -8,7 +8,21 @@
             </geometry>
             <origin xyz="0 0 0.05" rpy="0 0 0" />
+            <material name="blue" />
         </visual>
+        <collision>
+            <geometry>
+                <box size="0.56 0.385 0.335" />
+            </geometry>
+            <origin xyz="-0.0325 0.01 0.165" rpy="0 0 0" />
+        </collision>
+        <inertial>
+            <mass value="60.57865524" />
+            <origin xyz="-0.02389211 0.11375312 -0.00664723" rpy="0 0 0" />
+            <inertia ixx="1.12548060" ixy="-0.00628401" ixz="-0.04074518"
+                    iyy="3.07956336" iyz="0.00028181"
+                    izz="2.63020163" />
+        </inertial>
     </link>
-    <xacro:macro name="thruster_link" params="prefix x y z p" >
+    <xacro:macro name="thruster_link" params="prefix x y z p cp" >
         <link name="${prefix}_thruster_link">
             <visual>
@@ -17,13 +31,27 @@
                 </geometry>
                 <origin xyz="${x} ${y} ${z}" rpy="0 ${p} 0" />
+                <material name="grey" />
             </visual>
+            <collision>
+                <geometry>
+                    <cylinder radius="0.065" length="0.178" />
+                </geometry>
+                <origin xyz="0 0 0" rpy="0 ${cp} 0" />
+            </collision>
+            <inertial>
+                <mass value="1.59521765" />
+                <origin xyz="0.09333322 -0.00629336 -0.00002714" rpy="0 0 0" />
+                <inertia ixx="0.00101028" ixy="-0.00019770" ixz="0.00000211"
+                        iyy="0.00434934" iyz="-0.00000027"
+                        izz="0.00462580" />
+            </inertial>
         </link>
     </xacro:macro>
-    <xacro:thruster_link prefix="right_horizontal" x="0.025" y="-0.135" z="-0.235" p="0" />
-    <xacro:thruster_link prefix="left_horizontal" x="0.025" y="-0.135" z="-0.235" p="0" />
-    <xacro:thruster_link prefix="back_right_vertical" x="-0.03" y="-0.135" z="-0.235" p="0.26" />
-    <xacro:thruster_link prefix="back_left_vertical" x="0.09" y="-0.135" z="-0.235" p="-0.26" />
-    <xacro:thruster_link prefix="front_left_vertical" x="-0.03" y="-0.135" z="-0.235" p="0.26" />
-    <xacro:thruster_link prefix="front_right_vertical" x="0.09" y="-0.135" z="-0.235" p="-0.26" />
+    <xacro:thruster_link prefix="right_horizontal" x="0.025" y="-0.135" z="-0.235" p="0" cp="1.57" />
+    <xacro:thruster_link prefix="left_horizontal" x="0.025" y="-0.135" z="-0.235" p="0" cp="1.57" />
+    <xacro:thruster_link prefix="back_right_vertical" x="-0.03" y="-0.135" z="-0.235" p="0.26" cp="1.8326" />
+    <xacro:thruster_link prefix="back_left_vertical" x="0.09" y="-0.135" z="-0.235" p="-0.26" cp="-1.8326"/>
+    <xacro:thruster_link prefix="front_left_vertical" x="-0.03" y="-0.135" z="-0.235" p="0.26" cp="1.8326"/>
+    <xacro:thruster_link prefix="front_right_vertical" x="0.09" y="-0.135" z="-0.235" p="-0.26" cp="-1.8326"/>
     <xacro:macro name="thruster_propeller_link" params="prefix x" >
         <link name="${prefix}_thruster_propeller_link">
@@ -33,5 +61,19 @@
                 </geometry>
                 <origin xyz="${x} 0 0" rpy="0 0 0" />
+                <material name="red" />
             </visual>
+            <collision>
+                <geometry>
+                    <cylinder radius="0.045" length="0.06" />
+                </geometry>
+                <origin xyz="0 0 0.02" rpy="0 0 0" />
+            </collision>
+            <inertial>
+                <mass value="0.12426508" />
+                <origin xyz="0.00000013 0.02194882 -0.00000005" rpy="0 0 0" />
+                <inertia ixx="0.00002949" ixy="-0.00000000" ixz="-0.00000000"
+                        iyy="0.00001860" iyz="-0.00000000"
+                        izz="0.00002949" />
+            </inertial>
         </link>
     </xacro:macro>

Commit message: mods

File: reconbot_description/urdf/reconbot_mobile_base.xacro (robot description, xacro)
@@ -7,12 +7,12 @@
                 <mesh filename="package://reconbot_description/meshes/ReconBot_Main_Body.dae" />
             </geometry>
-            <origin xyz="0 0 0.05" rpy="0 0 0" />
+            <origin xyz="0 0 0.1" rpy="0 0 0" />
             <material name="blue" />
         </visual>
         <collision>
             <geometry>
-                <box size="0.56 0.385 0.335" />
+                <box size="0.62 0.380 0.32" />
             </geometry>
-            <origin xyz="-0.0325 0.01 0.165" rpy="0 0 0" />
+            <origin xyz="0 0 0.2" rpy="0 0 0" />
         </collision>
         <inertial>
@@ -23,6 +23,19 @@
                     izz="2.346243207" />
         </inertial>
+        <!-- Buoyancy Plugin -->
+        <plugin name='buoyancy' filename='libBuoyancyPlugin.so'>
+            <fluid_density>999.1026</fluid_density>
+            <center_of_volume>-0.0239 0.114 -0.007</center_of_volume>
+            <volume>0.00959081</volume>
+            <neutrally_buoyant>0</neutrally_buoyant>
+        </plugin>
+        <!-- Hydrodynamics Plugin -->
+        <plugin name='hydrodynamics_plugin' filename='libHydrodynamicsPlugin.so'>
+            <fluid_density>999.1026</fluid_density>
+            <linear_drag_coefficients>10.0 10.0 10.0</linear_drag_coefficients>
+            <angular_drag_coefficients>1.0 1.0 1.0</angular_drag_coefficients>
+        </plugin>
     </link>
-    <xacro:macro name="thruster_link" params="prefix x y z p cp" >
+    <xacro:macro name="thruster_link" params="prefix x y z p cx cp" >
         <link name="${prefix}_thruster_link">
             <visual>
@@ -37,5 +50,5 @@
                     <cylinder radius="0.065" length="0.178" />
                 </geometry>
-                <origin xyz="0 0 0" rpy="0 ${cp} 0" />
+                <origin xyz="${cx} 0 0" rpy="0 ${cp} 0" />
             </collision>
             <inertial>
@@ -48,10 +61,10 @@
         </link>
     </xacro:macro>
-    <xacro:thruster_link prefix="right_horizontal" x="0.025" y="-0.135" z="-0.235" p="0" cp="1.57" />
-    <xacro:thruster_link prefix="left_horizontal" x="0.025" y="-0.135" z="-0.235" p="0" cp="1.57" />
-    <xacro:thruster_link prefix="back_right_vertical" x="-0.03" y="-0.135" z="-0.235" p="0.26" cp="1.8326" />
-    <xacro:thruster_link prefix="back_left_vertical" x="0.09" y="-0.135" z="-0.235" p="-0.26" cp="-1.8326"/>
-    <xacro:thruster_link prefix="front_left_vertical" x="-0.03" y="-0.135" z="-0.235" p="0.26" cp="1.8326"/>
-    <xacro:thruster_link prefix="front_right_vertical" x="0.09" y="-0.135" z="-0.235" p="-0.26" cp="-1.8326"/>
+    <xacro:thruster_link prefix="right_horizontal" x="0.025" y="-0.135" z="-0.235" p="0" cx="0" cp="1.57" />
+    <xacro:thruster_link prefix="left_horizontal" x="0.025" y="-0.135" z="-0.235" p="0" cx="0" cp="1.57" />
+    <xacro:thruster_link prefix="back_right_vertical" x="-0.08" y="-0.135" z="-0.235" p="0.26" cx="-0.05" cp="1.8326" />
+    <xacro:thruster_link prefix="back_left_vertical" x="0.04" y="-0.135" z="-0.235" p="-0.26" cx="-0.05" cp="-1.8326"/>
+    <xacro:thruster_link prefix="front_left_vertical" x="-0.08" y="-0.135" z="-0.235" p="0.26" cx="-0.05" cp="1.8326"/>
+    <xacro:thruster_link prefix="front_right_vertical" x="0.04" y="-0.135" z="-0.235" p="-0.26" cx="-0.05" cp="-1.8326"/>
     <xacro:macro name="thruster_propeller_link" params="prefix x" >
         <link name="${prefix}_thruster_propeller_link">
@@ -96,6 +109,6 @@
         </joint>
     </xacro:macro>
-    <xacro:thruster_joint prefix="right_horizontal" x="-0.025" y="0.135" z="0.285" r="0" p="0" yw="0" />
-    <xacro:thruster_joint prefix="left_horizontal" x="-0.025" y="-0.1175" z="0.292" r="3.14" p="0" yw="0" />
+    <xacro:thruster_joint prefix="right_horizontal" x="-0.025" y="0.135" z="0.335" r="0" p="0" yw="0" />
+    <xacro:thruster_joint prefix="left_horizontal" x="-0.025" y="-0.1175" z="0.342" r="3.14" p="0" yw="0" />
     <xacro:thruster_joint prefix="back_right_vertical" x="0.32" y="0.09" z="0.18" r="1.57" p="1.57" yw="0" />
     <xacro:thruster_joint prefix="back_left_vertical" x="0.32" y="-0.09" z="0.18" r="1.57" p="1.57" yw="0" />
@@ -112,7 +125,7 @@
     <xacro:thruster_propeller_joint prefix="right_horizontal" x="0.0955" y="0" z="0" p="1.57" />
     <xacro:thruster_propeller_joint prefix="left_horizontal" x="0.0955" y="0" z="0" p="1.57" />
-    <xacro:thruster_propeller_joint prefix="back_right_vertical" x="0.0985" y="0.0022" z="-0.022" p="1.8326" />
-    <xacro:thruster_propeller_joint prefix="back_left_vertical" x="0.0955" y="0.0022" z="0.0125" p="1.309" />
-    <xacro:thruster_propeller_joint prefix="front_left_vertical" x="0.0985" y="0.0022" z="-0.022" p="1.8326" />
-    <xacro:thruster_propeller_joint prefix="front_right_vertical" x="0.0955" y="0.0022" z="0.0125" p="1.309" />
+    <xacro:thruster_propeller_joint prefix="back_right_vertical" x="0.0485" y="0.0022" z="-0.022" p="1.8326" />
+    <xacro:thruster_propeller_joint prefix="back_left_vertical" x="0.0455" y="0.0022" z="0.0125" p="1.309" />
+    <xacro:thruster_propeller_joint prefix="front_left_vertical" x="0.0485" y="0.0022" z="-0.022" p="1.8326" />
+    <xacro:thruster_propeller_joint prefix="front_right_vertical" x="0.0455" y="0.0022" z="0.0125" p="1.309" />
 </robot>

File: reconbot_description/urdf/reconbot_mobile_base_gazebo.xacro (robot description, xacro)
@@ -40,6 +40,19 @@
         <material>Gazebo/Red</material>
     </gazebo>
-    <plugin name='buoyancy' filename='libBuoyancyPlugin.so'>
+    <!-- <plugin name='buoyancy_plugin' filename='libBuoyancyPlugin.so'>
+        <fluid_density>997</fluid_density>
+        <link name='base_link'>
+          <center_of_buoyancy>0 0 0.1</center_of_buoyancy>
+          <volume>100000</volume>
+          <neutrally_buoyant>0</neutrally_buoyant>
+        </link>
+      </plugin> -->
+    <!-- <gazebo>
+        <plugin name='hydrodynamics_plugin' filename='libHydrodynamicsPlugin.so'>
+        <link_name>base_link</link_name>
         <fluid_density>999.1026</fluid_density>
-    </plugin>
+        <linear_drag_coefficients>10.0 10.0 10.0</linear_drag_coefficients>
+        <angular_drag_coefficients>1.0 1.0 1.0</angular_drag_coefficients>
+        </plugin>
+    </gazebo> -->
 </robot>

Commit message: mods

File: reconbot_description/urdf/reconbot_mobile_base.xacro (robot description, xacro)
@@ -2,4 +2,12 @@
 <robot xmlns:xacro="http://www.ros.org/wiki/xacro">
     <link name="base_footprint" />
+    <!-- <link name="water_link">
+        <collision>
+            <geometry>
+                <box size="10 10 5" />
+            </geometry>
+            <origin xyz="0 0 0" rpy="0 0 0" />
+        </collision>
+    </link> -->
     <link name="base_link">
         <visual>
@@ -17,23 +25,11 @@
         </collision>
         <inertial>
-            <mass value="60.57865524" />
-            <origin xyz="0 0 0.1675" rpy="0 0 0" />
-            <inertia ixx="2.173711367" ixy="0" ixz="0"
-                    iyy="1.252410727" iyz="0"
-                    izz="2.346243207" />
+            <!-- <mass value="60.57865524" /> -->
+            <mass value="81.47" />
+            <origin xyz="0 0 0.2" rpy="0 0 0" />
+            <inertia ixx="1.12548060" ixy="-0.00628401" ixz="-0.04074518"
+                    iyy="3.07956336" iyz="0.0028181"
+                    izz="2.63020163" />
         </inertial>
-        <!-- Buoyancy Plugin -->
-        <plugin name='buoyancy' filename='libBuoyancyPlugin.so'>
-            <fluid_density>999.1026</fluid_density>
-            <center_of_volume>-0.0239 0.114 -0.007</center_of_volume>
-            <volume>0.00959081</volume>
-            <neutrally_buoyant>0</neutrally_buoyant>
-        </plugin>
-        <!-- Hydrodynamics Plugin -->
-        <plugin name='hydrodynamics_plugin' filename='libHydrodynamicsPlugin.so'>
-            <fluid_density>999.1026</fluid_density>
-            <linear_drag_coefficients>10.0 10.0 10.0</linear_drag_coefficients>
-            <angular_drag_coefficients>1.0 1.0 1.0</angular_drag_coefficients>
-        </plugin>
     </link>
     <xacro:macro name="thruster_link" params="prefix x y z p cx cp" >
@@ -54,8 +50,8 @@
             <inertial>
                 <mass value="1.59521765" />
-                <origin xyz="0 0 0.065" rpy="0 0 0" />
-                <inertia ixx="0.00706634094" ixy="0" ixz="0"
-                        iyy="0.00706634094" iyz="0"
-                        izz="0.00336989728" />
+                <origin xyz="0 0 0" rpy="0 0 0" />
+                <inertia ixx="0.00101028" ixy="-0.00019770" ixz="0.00000211"
+                        iyy="0.00434934" iyz="-0.00000027"
+                        izz="0.00462580" />
             </inertial>
         </link>
@@ -84,8 +80,8 @@
             <inertial>
                 <mass value="0.12426508" />
-                <origin xyz="0 0 0.045" rpy="0 0 0" />
-                <inertia ixx="0.00010018872" ixy="0" ixz="0"
-                        iyy="0.00010018872" iyz="0"
-                        izz="0.00012581839" />
+                <origin xyz="0 0 0" rpy="0 0 0" />
+                <inertia ixx="0.00002949" ixy="0" ixz="0"
+                        iyy="0.00001860" iyz="0"
+                        izz="0.00002949" />
             </inertial>
         </link>
@@ -97,4 +93,9 @@
     <xacro:thruster_propeller_link prefix="front_left_vertical" x="0" />
     <xacro:thruster_propeller_link prefix="front_right_vertical" x="0" />
+    <!-- <joint name="base_water_joint" type="fixed" >
+        <parent link="base_footprint" />
+        <child link="water_link" />
+        <origin xyz="0 0 0" rpy="0 0 0" />
+    </joint> -->
     <joint name="base_joint" type="fixed" >
         <parent link="base_footprint" />

File: reconbot_description/urdf/reconbot_mobile_base_gazebo.xacro (robot description, xacro)
@@ -40,19 +40,30 @@
         <material>Gazebo/Red</material>
     </gazebo>
-    <!-- <plugin name='buoyancy_plugin' filename='libBuoyancyPlugin.so'>
-        <fluid_density>997</fluid_density>
-        <link name='base_link'>
-          <center_of_buoyancy>0 0 0.1</center_of_buoyancy>
-          <volume>100000</volume>
-          <neutrally_buoyant>0</neutrally_buoyant>
-        </link>
-      </plugin> -->
-    <!-- <gazebo>
-        <plugin name='hydrodynamics_plugin' filename='libHydrodynamicsPlugin.so'>
-        <link_name>base_link</link_name>
-        <fluid_density>999.1026</fluid_density>
-        <linear_drag_coefficients>10.0 10.0 10.0</linear_drag_coefficients>
-        <angular_drag_coefficients>1.0 1.0 1.0</angular_drag_coefficients>
-        </plugin>
-    </gazebo> -->
+    <xacro:macro name="buoyancy_plugin_link" params="link volume cobx">
+        <gazebo>
+            <plugin name='buoyancy_plugin' filename='libBuoyancyPlugin.so'>
+                <fluid_density>999.1026</fluid_density>
+                <link name='${link}'>
+                <center_of_buoyancy>0 0 ${cobx}</center_of_buoyancy>
+                <volume>${volume}</volume>
+                <neutrally_buoyant>0</neutrally_buoyant>
+                </link>
+            </plugin>
+        </gazebo>
+        <gazebo>
+            <plugin name='hydrodynamics_plugin' filename='libHydrodynamicsPlugin.so'>
+            <link_name>${link}</link_name>
+            <fluid_density>999.1026</fluid_density>
+            <linear_drag_coefficients>10.0 10.0 10.0</linear_drag_coefficients>
+            <angular_drag_coefficients>1.0 1.0 1.0</angular_drag_coefficients>
+            </plugin>
+        </gazebo>
+    </xacro:macro>
+    <xacro:buoyancy_plugin_link link="base_link" volume="0.00959081" cobx="0.25" />
+    <!-- <xacro:buoyancy_plugin_link link="right_horizontal_thruster_link" volume="0.00031572" cobx="0" />
+    <xacro:buoyancy_plugin_link link="left_horizontal_thruster_link" volume="0.00031572" cobx="0" />
+    <xacro:buoyancy_plugin_link link="back_right_vertical_thruster_link" volume="0.00031572" cobx="0" />
+    <xacro:buoyancy_plugin_link link="back_left_vertical_thruster_link" volume="0.00031572" cobx="0" />
+    <xacro:buoyancy_plugin_link link="front_left_vertical_thruster_link" volume="0.00031572" cobx="0" />
+    <xacro:buoyancy_plugin_link link="front_right_vertical_thruster_link" volume="0.00031572" cobx="0" /> -->
 </robot>

Commit message: mods

File: reconbot_description/urdf/reconbot_mobile_base.xacro (robot description, xacro)
@@ -2,12 +2,4 @@
 <robot xmlns:xacro="http://www.ros.org/wiki/xacro">
     <link name="base_footprint" />
-    <!-- <link name="water_link">
-        <collision>
-            <geometry>
-                <box size="10 10 5" />
-            </geometry>
-            <origin xyz="0 0 0" rpy="0 0 0" />
-        </collision>
-    </link> -->
     <link name="base_link">
         <visual>
@@ -22,10 +14,10 @@
                 <box size="0.62 0.380 0.32" />
             </geometry>
-            <origin xyz="0 0 0.2" rpy="0 0 0" />
+            <origin xyz="-0.025 0 0.2" rpy="0 0 0" />
         </collision>
         <inertial>
             <!-- <mass value="60.57865524" /> -->
-            <mass value="81.47" />
-            <origin xyz="0 0 0.2" rpy="0 0 0" />
+            <mass value="81.46" />
+            <origin xyz="-0.025 0 0.2" rpy="0 0 0" />
             <inertia ixx="1.12548060" ixy="-0.00628401" ixz="-0.04074518"
                     iyy="3.07956336" iyz="0.0028181"
@@ -93,9 +85,4 @@
     <xacro:thruster_propeller_link prefix="front_left_vertical" x="0" />
     <xacro:thruster_propeller_link prefix="front_right_vertical" x="0" />
-    <!-- <joint name="base_water_joint" type="fixed" >
-        <parent link="base_footprint" />
-        <child link="water_link" />
-        <origin xyz="0 0 0" rpy="0 0 0" />
-    </joint> -->
     <joint name="base_joint" type="fixed" >
         <parent link="base_footprint" />

File: reconbot_description/urdf/reconbot_mobile_base_gazebo.xacro (robot description, xacro)
@@ -40,30 +40,21 @@
         <material>Gazebo/Red</material>
     </gazebo>
-    <xacro:macro name="buoyancy_plugin_link" params="link volume cobx">
-        <gazebo>
-            <plugin name='buoyancy_plugin' filename='libBuoyancyPlugin.so'>
-                <fluid_density>999.1026</fluid_density>
-                <link name='${link}'>
-                <center_of_buoyancy>0 0 ${cobx}</center_of_buoyancy>
-                <volume>${volume}</volume>
-                <neutrally_buoyant>0</neutrally_buoyant>
-                </link>
-            </plugin>
-        </gazebo>
-        <gazebo>
-            <plugin name='hydrodynamics_plugin' filename='libHydrodynamicsPlugin.so'>
-            <link_name>${link}</link_name>
+    <gazebo>
+        <plugin name='buoyancy_plugin' filename='libBuoyancyPlugin.so'>
             <fluid_density>999.1026</fluid_density>
-            <linear_drag_coefficients>10.0 10.0 10.0</linear_drag_coefficients>
-            <angular_drag_coefficients>1.0 1.0 1.0</angular_drag_coefficients>
-            </plugin>
-        </gazebo>
-    </xacro:macro>
-    <xacro:buoyancy_plugin_link link="base_link" volume="0.00959081" cobx="0.25" />
-    <!-- <xacro:buoyancy_plugin_link link="right_horizontal_thruster_link" volume="0.00031572" cobx="0" />
-    <xacro:buoyancy_plugin_link link="left_horizontal_thruster_link" volume="0.00031572" cobx="0" />
-    <xacro:buoyancy_plugin_link link="back_right_vertical_thruster_link" volume="0.00031572" cobx="0" />
-    <xacro:buoyancy_plugin_link link="back_left_vertical_thruster_link" volume="0.00031572" cobx="0" />
-    <xacro:buoyancy_plugin_link link="front_left_vertical_thruster_link" volume="0.00031572" cobx="0" />
-    <xacro:buoyancy_plugin_link link="front_right_vertical_thruster_link" volume="0.00031572" cobx="0" /> -->
+            <link name='base_link'>
+            <center_of_buoyancy>-0.025 0 0.25</center_of_buoyancy>
+            <volume>0.00959081</volume>
+            <neutrally_buoyant>0</neutrally_buoyant>
+            </link>
+        </plugin>
+    </gazebo>
+    <gazebo>
+        <plugin name='hydrodynamics_plugin' filename='libHydrodynamicsPlugin.so'>
+        <link_name>base_link</link_name>
+        <fluid_density>999.1026</fluid_density>
+        <linear_drag_coefficients>10.0 10.0 10.0</linear_drag_coefficients>
+        <angular_drag_coefficients>1.0 1.0 1.0</angular_drag_coefficients>
+        </plugin>
+    </gazebo>
 </robot>

Commit message: imu addition

File: reconbot_description/urdf/reconbot_mobile_base.xacro (robot description, xacro)
@@ -109,4 +109,6 @@
             <origin xyz="${x} ${y} ${z}" rpy="0 ${p} 0" />
             <axis xyz="0 0 1" />
+            <!-- <limit effort="100" velocity="0"/> -->
+            <!-- <dynamics damping="0.1" friction="0.1"/> -->
         </joint>
     </xacro:macro>

File: reconbot_description/urdf/reconbot_mobile_base_gazebo.xacro (robot description, xacro)
@@ -58,3 +58,23 @@
         </plugin>
     </gazebo>
+      <gazebo reference="base_link">
+        <gravity>true</gravity>
+        <sensor name="imu_sensor" type="imu">
+        <always_on>true</always_on>
+        <update_rate>100</update_rate>
+        <visualize>true</visualize>
+        <topic>__default_topic__</topic>
+        <plugin filename="libgazebo_ros_imu_sensor.so" name="imu_plugin">
+            <topicName>imu</topicName>
+            <bodyName>base_link</bodyName>
+            <updateRateHZ>10.0</updateRateHZ>
+            <gaussianNoise>0.0</gaussianNoise>
+            <xyzOffset>0 0 0</xyzOffset>
+            <rpyOffset>0 0 0</rpyOffset>
+            <frameName>base_link</frameName>
+            <initialOrientationAsReference>false</initialOrientationAsReference>
+        </plugin>
+        <pose>0 0 0 0 0 0</pose>
+        </sensor>
+    </gazebo>
 </robot>
