Commit message: reconbot addition

File: gr2_description/urdf/gr2_mobile_base.xacro (robot description, xacro)
@@ -6,6 +6,38 @@
             <geometry>
                 <mesh filename="package://gr2_description/meshes/GR2_Main_Body.dae" />
-                <origin xyz="0 0 0" rpy="0 0 0" />
             </geometry>
+            <origin xyz="0.08 0 0" rpy="0 0 0" />
+        </visual>
+    </link>
+    <link name="left_front_wheel_link">
+        <visual>
+            <geometry>
+                <mesh filename="package://gr2_description/meshes/GR2_Wheel_Assembly.dae" />
+            </geometry>
+            <origin xyz="0 0 0" rpy="0 0 0" />
+        </visual>
+    </link>
+    <link name="right_front_wheel_link">
+        <visual>
+            <geometry>
+                <mesh filename="package://gr2_description/meshes/GR2_Wheel_Assembly.dae" />
+            </geometry>
+            <origin xyz="0 0 0" rpy="0 0 0" />
+        </visual>
+    </link>
+    <link name="right_back_wheel_link">
+        <visual>
+            <geometry>
+                <mesh filename="package://gr2_description/meshes/GR2_Wheel_Assembly.dae" />
+            </geometry>
+            <origin xyz="0 0 0" rpy="0 0 0" />
+        </visual>
+    </link>
+    <link name="left_back_wheel_link">
+        <visual>
+            <geometry>
+                <mesh filename="package://gr2_description/meshes/GR2_Wheel_Assembly.dae" />
+            </geometry>
+            <origin xyz="0 0 0" rpy="0 0 0" />
         </visual>
     </link>
@@ -15,3 +47,27 @@
         <origin xyz="0 0 0.015" rpy="0 0 0" />
     </joint>
+    <joint name="left_front_wheel_joint" type="continuous" >
+        <parent link="base_link" />
+        <child link="left_front_wheel_link" />
+        <origin xyz="0.09 -0.075 0.0" rpy="0 0 1.57" />
+        <axis xyz="0 1 0" />
+    </joint>
+    <joint name="right_front_wheel_joint" type="continuous" >
+        <parent link="base_link" />
+        <child link="right_front_wheel_link" />
+        <origin xyz="-0.088 -0.075 0.0" rpy="0 0 -1.57" />
+        <axis xyz="0 1 0" />
+    </joint>
+    <joint name="right_back_wheel_joint" type="continuous" >
+        <parent link="base_link" />
+        <child link="right_back_wheel_link" />
+        <origin xyz="-0.088 0.052 0.0" rpy="0 0 -1.57" />
+        <axis xyz="0 1 0" />
+    </joint>
+    <joint name="left_back_wheel_joint" type="continuous" >
+        <parent link="base_link" />
+        <child link="left_back_wheel_link" />
+        <origin xyz="0.088 0.052 0.0" rpy="0 0 1.57" />
+        <axis xyz="0 1 0" />
+    </joint>
 </robot>

Commit message: gr2 control

File: gr2_description/urdf/gr2_mobile_base.xacro (robot description, xacro)
@@ -1,4 +1,4 @@
 <?xml version="1.0"?>
-<robot name="gr2" xmlns:xacro="http://www.ros.org/wiki/xacro">
+<robot xmlns:xacro="http://www.ros.org/wiki/xacro">
     <link name="base_footprint" />
     <link name="base_link">
@@ -8,66 +8,64 @@
             </geometry>
             <origin xyz="0.08 0 0" rpy="0 0 0" />
+            <material name="grey" />
         </visual>
+        <collision>
+            <geometry>
+                <box size="0.140 0.160 0.143" />
+            </geometry>
+            <origin xyz="0.0015 -0.015 0.055" rpy="0 0 0" />
+        </collision>
+        <inertial>
+            <mass value="0.715" />
+            <origin xyz="0 0 0" rpy="0 0 0" />
+            <inertia ixx="0.003" ixy="6.408e-5" ixz="-6.085e-5"
+                    iyy="0.002" iyz="-1.701e-6"
+                    izz="0.003" />
+        </inertial>
     </link>
-    <link name="left_front_wheel_link">
-        <visual>
-            <geometry>
-                <mesh filename="package://gr2_description/meshes/GR2_Wheel_Assembly.dae" />
-            </geometry>
-            <origin xyz="0 0 0" rpy="0 0 0" />
-        </visual>
-    </link>
-    <link name="right_front_wheel_link">
-        <visual>
-            <geometry>
-                <mesh filename="package://gr2_description/meshes/GR2_Wheel_Assembly.dae" />
-            </geometry>
-            <origin xyz="0 0 0" rpy="0 0 0" />
-        </visual>
-    </link>
-    <link name="right_back_wheel_link">
-        <visual>
-            <geometry>
-                <mesh filename="package://gr2_description/meshes/GR2_Wheel_Assembly.dae" />
-            </geometry>
-            <origin xyz="0 0 0" rpy="0 0 0" />
-        </visual>
-    </link>
-    <link name="left_back_wheel_link">
-        <visual>
-            <geometry>
-                <mesh filename="package://gr2_description/meshes/GR2_Wheel_Assembly.dae" />
-            </geometry>
-            <origin xyz="0 0 0" rpy="0 0 0" />
-        </visual>
-    </link>
+    <xacro:macro name="wheel_link" params="prefix" >
+        <link name="${prefix}_wheel_link">
+            <visual>
+                <geometry>
+                    <mesh filename="package://gr2_description/meshes/GR2_Wheel_Assembly.dae" />
+                </geometry>
+                <origin xyz="0 0 0" rpy="0 0 0" />
+                <material name="blue" />
+            </visual>
+            <collision>
+                <geometry>
+                    <cylinder radius="0.031" length="0.047" />
+                </geometry>
+                <origin xyz="0 0 0" rpy="1.57 0 0" />
+            </collision>
+            <inertial>
+                <mass value="0.062" />
+                <origin xyz="0 0 0" rpy="0 0 0" />
+                <inertia ixx="2.527e-5" ixy="4.039e-11" ixz="2.637e-12"
+                        iyy="1.528e-5" iyz="9.797e-11"
+                        izz="1.528e-5" />
+            </inertial>
+        </link>
+    </xacro:macro>
+    <xacro:wheel_link prefix="left_front" />
+    <xacro:wheel_link prefix="right_front" />
+    <xacro:wheel_link prefix="left_back" />
+    <xacro:wheel_link prefix="right_back" />
     <joint name="base_joint" type="fixed" >
         <parent link="base_footprint" />
         <child link="base_link" />
-        <origin xyz="0 0 0.015" rpy="0 0 0" />
+        <origin xyz="0 0 0.05" rpy="0 0 0" />
     </joint>
-    <joint name="left_front_wheel_joint" type="continuous" >
-        <parent link="base_link" />
-        <child link="left_front_wheel_link" />
-        <origin xyz="0.09 -0.075 0.0" rpy="0 0 1.57" />
-        <axis xyz="0 1 0" />
-    </joint>
-    <joint name="right_front_wheel_joint" type="continuous" >
-        <parent link="base_link" />
-        <child link="right_front_wheel_link" />
-        <origin xyz="-0.088 -0.075 0.0" rpy="0 0 -1.57" />
-        <axis xyz="0 1 0" />
-    </joint>
-    <joint name="right_back_wheel_joint" type="continuous" >
-        <parent link="base_link" />
-        <child link="right_back_wheel_link" />
-        <origin xyz="-0.088 0.052 0.0" rpy="0 0 -1.57" />
-        <axis xyz="0 1 0" />
-    </joint>
-    <joint name="left_back_wheel_joint" type="continuous" >
-        <parent link="base_link" />
-        <child link="left_back_wheel_link" />
-        <origin xyz="0.088 0.052 0.0" rpy="0 0 1.57" />
-        <axis xyz="0 1 0" />
-    </joint>
+    <xacro:macro name="wheel_joint" params="prefix x y yw ay" >
+        <joint name="base_${prefix}_wheel_joint" type="continuous" >
+            <parent link="base_link" />
+            <child link="${prefix}_wheel_link" />
+            <origin xyz="${x} ${y} 0.0" rpy="0 0 ${yw}" />
+            <axis xyz="0 ${ay} 0" />
+        </joint>
+    </xacro:macro>
+    <xacro:wheel_joint prefix="left_front" x="0.09" y="-0.075" yw="1.57" ay="-1" />
+    <xacro:wheel_joint prefix="right_front" x="-0.088" y="-0.075" yw="-1.57" ay="1" />
+    <xacro:wheel_joint prefix="left_back" x="0.088" y="0.052" yw="1.57" ay="-1" />
+    <xacro:wheel_joint prefix="right_back" x="-0.088" y="0.052" yw="-1.57" ay="1" />
 </robot>

File: reconbot_description/urdf/reconbot_mobile_base.xacro (robot description, xacro)
@@ -109,6 +109,4 @@
             <origin xyz="${x} ${y} ${z}" rpy="0 ${p} 0" />
             <axis xyz="0 0 1" />
-            <!-- <limit effort="100" velocity="0"/> -->
-            <!-- <dynamics damping="0.1" friction="0.1"/> -->
         </joint>
     </xacro:macro>
@@ -119,3 +117,13 @@
     <xacro:thruster_propeller_joint prefix="front_left_vertical" x="0.0485" y="0.0022" z="-0.022" p="1.8326" />
     <xacro:thruster_propeller_joint prefix="front_right_vertical" x="0.0455" y="0.0022" z="0.0125" p="1.309" />
+     <!-- Transmission for the thruster -->
+    <transmission name="right_horizontal_thruster_propeller_trans">
+        <type>transmission_interface/SimpleTransmission</type>
+        <joint name="right_horizontal_thruster_propeller_joint">
+        <hardwareInterface>hardware_interface/EffortJointInterface</hardwareInterface>
+        </joint>
+        <actuator name="right_horizontal_thruster">
+        <mechanicalReduction>1</mechanicalReduction>
+        </actuator>
+    </transmission>
 </robot>

File: reconbot_description/urdf/reconbot_mobile_base_gazebo.xacro (robot description, xacro)
@@ -78,9 +78,14 @@
         </sensor>
     </gazebo>
-    <gazebo>
+    <!-- <gazebo>
         <plugin name="rov_interface_plugin" filename="librov_interface_plugin.so">
             <left_horizontal_propeller_joint>left_horizontal_propeller_joint</left_horizontal_propeller_joint>
             <right_horizontal_propeller_joint>right_horizontal_propeller_joint</right_horizontal_propeller_joint>
         </plugin>
+    </gazebo> -->
+    <gazebo>
+        <plugin name="gazebo_ros_control" filename="libgazebo_ros_control.so">
+            <robotNamespace>/reconbot</robotNamespace>
+        </plugin>
     </gazebo>
 </robot>

Commit message: mods

File: gr2_description/urdf/gr2_mobile_base.xacro (robot description, xacro)
@@ -52,4 +52,26 @@
     <xacro:wheel_link prefix="left_back" />
     <xacro:wheel_link prefix="right_back" />
+    <link name="camera_link">
+        <visual>
+            <geometry>
+                <mesh filename="package://gr2_description/meshes/GR2_Cam_Mount.dae" />
+            </geometry>
+            <origin xyz="0 0 0" rpy="0 0 0" />
+            <material name="grey" />
+        </visual>
+        <collision>
+            <geometry>
+                <box size="0.044 0.057 0.04" />
+            </geometry>
+            <origin xyz="0.0105 0.0125 0.0115" rpy="0 0 0" />
+        </collision>
+        <inertial>
+            <mass value="0.014" />
+            <origin xyz="0 0 0" rpy="0 0 0" />
+            <inertia ixx="3.888e-6" ixy="-6.953e-9" ixz="8.281e-9"
+                    iyy="3.246e-6" iyz="1.170e-6"
+                    izz="3.570e-6" />
+        </inertial>
+    </link>
     <joint name="base_joint" type="fixed" >
         <parent link="base_footprint" />
@@ -69,3 +91,8 @@
     <xacro:wheel_joint prefix="left_back" x="0.088" y="0.052" yw="1.57" ay="-1" />
     <xacro:wheel_joint prefix="right_back" x="-0.088" y="0.052" yw="-1.57" ay="1" />
+    <joint name="base_camera_joint" type="fixed">
+        <parent link="base_link"/>
+        <child link="camera_link"/>
+        <origin xyz="-0.01 -0.1045 0.028" rpy="0 0 0" />
+    </joint>
 </robot>

File: gr2_description/urdf/gr2_mobile_base_gazebo.xacro (robot description, xacro)
@@ -48,3 +48,43 @@
         </plugin>
     </gazebo>
+    <!-- camera -->
+    <gazebo reference="camera_link">
+        <sensor type="camera" name="camera1">
+        <update_rate>30.0</update_rate>
+        <camera name="head">
+            <horizontal_fov>1.3962634</horizontal_fov>
+            <image>
+            <width>800</width>
+            <height>800</height>
+            <format>R8G8B8</format>
+            </image>
+            <clip>
+            <near>0.02</near>
+            <far>300</far>
+            </clip>
+            <noise>
+            <type>gaussian</type>
+            <!-- Noise is sampled independently per pixel on each frame.
+                That pixel's noise value is added to each of its color
+                channels, which at that point lie in the range [0,1]. -->
+            <mean>0.0</mean>
+            <stddev>0.007</stddev>
+            </noise>
+        </camera>
+        <plugin name="camera_controller" filename="libgazebo_ros_camera.so">
+            <alwaysOn>true</alwaysOn>
+            <updateRate>0.0</updateRate>
+            <cameraName>gr2/camera1</cameraName>
+            <imageTopicName>image_raw</imageTopicName>
+            <cameraInfoTopicName>camera_info</cameraInfoTopicName>
+            <frameName>camera_link</frameName>
+            <hackBaseline>0.07</hackBaseline>
+            <distortionK1>0.0</distortionK1>
+            <distortionK2>0.0</distortionK2>
+            <distortionK3>0.0</distortionK3>
+            <distortionT1>0.0</distortionT1>
+            <distortionT2>0.0</distortionT2>
+        </plugin>
+        </sensor>
+    </gazebo>
 </robot>

File: reconbot_description/urdf/reconbot_mobile_base.xacro (robot description, xacro)
@@ -25,5 +25,5 @@
         </inertial>
     </link>
-    <xacro:macro name="thruster_link" params="prefix x y z p cx cp" >
+    <xacro:macro name="thruster_link" params="prefix x y z p cx cp ix iz" >
         <link name="${prefix}_thruster_link">
             <visual>
@@ -42,5 +42,5 @@
             <inertial>
                 <mass value="1.59521765" />
-                <origin xyz="0 0 0" rpy="0 0 0" />
+                <origin xyz="${ix} 0 ${iz}" rpy="0 0 0" />
                 <inertia ixx="0.00101028" ixy="-0.00019770" ixz="0.00000211"
                         iyy="0.00434934" iyz="-0.00000027"
@@ -49,10 +49,10 @@
         </link>
     </xacro:macro>
-    <xacro:thruster_link prefix="right_horizontal" x="0.025" y="-0.135" z="-0.235" p="0" cx="0" cp="1.57" />
-    <xacro:thruster_link prefix="left_horizontal" x="0.025" y="-0.135" z="-0.235" p="0" cx="0" cp="1.57" />
-    <xacro:thruster_link prefix="back_right_vertical" x="-0.08" y="-0.135" z="-0.235" p="0.26" cx="-0.05" cp="1.8326" />
-    <xacro:thruster_link prefix="back_left_vertical" x="0.04" y="-0.135" z="-0.235" p="-0.26" cx="-0.05" cp="-1.8326"/>
-    <xacro:thruster_link prefix="front_left_vertical" x="-0.08" y="-0.135" z="-0.235" p="0.26" cx="-0.05" cp="1.8326"/>
-    <xacro:thruster_link prefix="front_right_vertical" x="0.04" y="-0.135" z="-0.235" p="-0.26" cx="-0.05" cp="-1.8326"/>
+    <xacro:thruster_link prefix="right_horizontal" x="0.025" y="-0.135" z="-0.235" p="0" cx="0" cp="1.57" ix="0" iz="0" />
+    <xacro:thruster_link prefix="left_horizontal" x="0.025" y="-0.135" z="-0.235" p="0" cx="0" cp="1.57" ix="0" iz="0" />
+    <xacro:thruster_link prefix="back_right_vertical" x="-0.08" y="-0.135" z="-0.235" p="0.26" cx="-0.05" cp="1.8326" ix="-0.05" iz="0" />
+    <xacro:thruster_link prefix="back_left_vertical" x="0.04" y="-0.135" z="-0.235" p="-0.26" cx="-0.05" cp="-1.8326" ix="-0.05" iz="-0.01" />
+    <xacro:thruster_link prefix="front_left_vertical" x="-0.08" y="-0.135" z="-0.235" p="0.26" cx="-0.05" cp="1.8326" ix="-0.05" iz="0" />
+    <xacro:thruster_link prefix="front_right_vertical" x="0.04" y="-0.135" z="-0.235" p="-0.26" cx="-0.05" cp="-1.8326" ix="-0.05" iz="-0.01" />
     <xacro:macro name="thruster_propeller_link" params="prefix x" >
         <link name="${prefix}_thruster_propeller_link">
@@ -72,5 +72,5 @@
             <inertial>
                 <mass value="0.12426508" />
-                <origin xyz="0 0 0" rpy="0 0 0" />
+                <origin xyz="0 0 0.025" rpy="0 0 0" />
                 <inertia ixx="0.00002949" ixy="0" ixz="0"
                         iyy="0.00001860" iyz="0"
@@ -118,12 +118,13 @@
     <xacro:thruster_propeller_joint prefix="front_right_vertical" x="0.0455" y="0.0022" z="0.0125" p="1.309" />
      <!-- Transmission for the thruster -->
-    <!-- <transmission name="right_horizontal_thruster_propeller_trans">
+    <transmission name="right_horizontal_thruster_propeller_trans">
         <type>transmission_interface/SimpleTransmission</type>
         <joint name="right_horizontal_thruster_propeller_joint">
-        <hardwareInterface>hardware_interface/EffortJointInterface</hardwareInterface>
+            <hardwareInterface>EffortJointInterface</hardwareInterface>
         </joint>
         <actuator name="right_horizontal_thruster">
-        <mechanicalReduction>1</mechanicalReduction>
+            <mechanicalReduction>1</mechanicalReduction>
+            <hardwareInterface>EffortJointInterface</hardwareInterface>
         </actuator>
-    </transmission> -->
+    </transmission>
 </robot>

File: reconbot_description/urdf/reconbot_mobile_base_gazebo.xacro (robot description, xacro)
@@ -44,7 +44,7 @@
             <fluid_density>999.1026</fluid_density>
             <link name='base_link'>
-            <center_of_buoyancy>-0.025 0 0.25</center_of_buoyancy>
-            <volume>0.00959081</volume>
-            <neutrally_buoyant>0</neutrally_buoyant>
+                <center_of_buoyancy>-0.025 0 0.25</center_of_buoyancy>
+                <volume>0.00959081</volume>
+                <neutrally_buoyant>0</neutrally_buoyant>
             </link>
         </plugin>
@@ -52,11 +52,11 @@
     <gazebo>
         <plugin name='hydrodynamics_plugin' filename='libHydrodynamicsPlugin.so'>
-        <link_name>base_link</link_name>
-        <fluid_density>999.1026</fluid_density>
-        <linear_drag_coefficients>10.0 10.0 10.0</linear_drag_coefficients>
-        <angular_drag_coefficients>1.0 1.0 1.0</angular_drag_coefficients>
+            <link_name>base_link</link_name>
+            <fluid_density>999.1026</fluid_density>
+            <linear_drag_coefficients>10.0 10.0 10.0</linear_drag_coefficients>
+            <angular_drag_coefficients>1.0 1.0 1.0</angular_drag_coefficients>
         </plugin>
     </gazebo>
-      <gazebo reference="base_link">
+    <!-- <gazebo reference="base_link">
         <gravity>true</gravity>
         <sensor name="imu_sensor" type="imu">
@@ -77,5 +77,5 @@
         <pose>0 0 0 0 0 0</pose>
         </sensor>
-    </gazebo>
+    </gazebo> -->
     <!-- <gazebo>
         <plugin name="rov_interface_plugin" filename="librov_interface_plugin.so">
@@ -84,8 +84,8 @@
         </plugin>
     </gazebo> -->
-    <!-- <gazebo>
+    <gazebo>
         <plugin name="gazebo_ros_control" filename="libgazebo_ros_control.so">
             <robotNamespace>/reconbot</robotNamespace>
         </plugin>
-    </gazebo> -->
+    </gazebo>
 </robot>

Commit message: robot_localization

File: gr2_description/urdf/gr2_mobile_base.xacro (robot description, xacro)
@@ -57,5 +57,5 @@
                 <mesh filename="package://gr2_description/meshes/GR2_Cam_Mount.dae" />
             </geometry>
-            <origin xyz="0 0 0" rpy="0 0 0" />
+            <origin xyz="0 0 0" rpy="0 0 1.57" />
             <material name="grey" />
         </visual>
@@ -94,5 +94,5 @@
         <parent link="base_link"/>
         <child link="camera_link"/>
-        <origin xyz="-0.01 -0.1045 0.028" rpy="0 0 0" />
+        <origin xyz="-0.01 -0.1045 0.028" rpy="0 0 4.71" />
     </joint>
 </robot>

File: gr2_description/urdf/gr2_mobile_base_gazebo.xacro (robot description, xacro)
@@ -22,4 +22,8 @@
     <gazebo>
         <plugin name="diff_drive_controller" filename="libgazebo_ros_diff_drive.so">
+            <ros>
+                <namespace>/robot</namespace>
+                <remapping>odom:=/odom</remapping>
+            </ros>
             <!-- Update rate in Hz -->
             <update_rate>50</update_rate>
@@ -35,6 +39,6 @@
             <wheel_diameter>0.062</wheel_diameter>
             <!-- limits -->
-            <!-- <max_wheel_torque>20</max_wheel_torque>
-            <max_wheel_acceleration>1.0</max_wheel_acceleration> -->
+            <max_wheel_torque>20</max_wheel_torque>
+            <max_wheel_acceleration>1.0</max_wheel_acceleration>
             <!-- input -->
             <command_topic>cmd_vel</command_topic>
@@ -88,3 +92,23 @@
         </sensor>
     </gazebo>
+    <gazebo reference="base_link">
+        <gravity>true</gravity>
+        <sensor name="imu_sensor" type="imu">
+        <always_on>true</always_on>
+        <update_rate>100</update_rate>
+        <visualize>true</visualize>
+        <topic>__default_topic__</topic>
+        <plugin filename="libgazebo_ros_imu_sensor.so" name="imu_plugin">
+            <topicName>imu</topicName>
+            <bodyName>base_link</bodyName>
+            <updateRateHZ>10.0</updateRateHZ>
+            <gaussianNoise>0.0</gaussianNoise>
+            <xyzOffset>0 0 0</xyzOffset>
+            <rpyOffset>0 0 0</rpyOffset>
+            <frameName>base_link</frameName>
+            <initialOrientationAsReference>true</initialOrientationAsReference>
+        </plugin>
+        <pose>0 0 0 0 0 0</pose>
+        </sensor>
+    </gazebo>
 </robot>
